File: PCB/Ganjing keyboard/Ganjing keyboard.sch (KiCad schematic (older format))
At the start: 166 parts, among them J1 Conn_01x04, J2 AVR-ISP-6, SW1 Rotary_Encoder_Switch, U1 ATmega32A-PU, Y1 Crystal

Commit message: Rearranging pins on MCU
Connections:
- net labels added: col5, col7, col9
- net labels removed: Col0, Col1, Col10, Col11, Col12, Col13, Col14, Col2, Col3, Col4, Col5, Col6, Col7, Col8, Col9, Row0, Row1, Row2, Row3, Row4
Changed lines of the file:
@@
 	1    0    0    -1
 $EndComp
-Text GLabel 2650 3650 2    50   Input ~ 0
+Text GLabel 2650 1450 2    50   Input ~ 0
 row3
+Text GLabel 2650 1550 2    50   Input ~ 0
+row1
+Text GLabel 2650 1650 2    50   Input ~ 0
+col0
+Text GLabel 2650 1750 2    50   Input ~ 0
+col2
+Text GLabel 2650 1850 2    50   Input ~ 0
+col4
+Text GLabel 2650 2650 2    50   Input ~ 0
+row2
+Text GLabel 2650 2750 2    50   Input ~ 0
+row0
+Text GLabel 2650 3450 2    50   Input ~ 0
+col1
 Text GLabel 2650 3550 2    50   Input ~ 0
-row1
-Text GLabel 2650 1450 2    50   Input ~ 0
-col0
-Text GLabel 2650 1550 2    50   Input ~ 0
-col2
-Text GLabel 2650 1650 2    50   Input ~ 0
-col4
-Text GLabel 2650 2350 2    50   Input ~ 0
-row4
-Text GLabel 2650 3950 2    50   Input ~ 0
-row2
-Text GLabel 2650 3450 2    50   Input ~ 0
-row0
-Text GLabel 2650 2650 2    50   Input ~ 0
-col1
-Text GLabel 2650 2750 2    50   Input ~ 0
 col3
 Text GLabel 2650 2450 2    50   Input ~ 0
@@
 Text GLabel 2650 2550 2    50   Input ~ 0
 B2
-Text GLabel 2650 1750 2    50   Input ~ 0
+Text GLabel 2650 1950 2    50   Input ~ 0
 col6
-Text GLabel 2650 1850 2    50   Input ~ 0
+Text GLabel 2650 2050 2    50   Input ~ 0
 col8
-Text GLabel 2650 1950 2    50   Input ~ 0
+Text GLabel 2650 2150 2    50   Input ~ 0
 col10
-Text GLabel 2650 2050 2    50   Input ~ 0
+Text GLabel 2650 3950 2    50   Input ~ 0
 col11
-Text GLabel 2650 2150 2    50   Input ~ 0
+Text GLabel 2650 4650 2    50   Input ~ 0
 col12
-Text GLabel 2650 3850 2    50   Input ~ 0
+Text GLabel 2650 2350 2    50   Input ~ 0
 row4
 Text GLabel 2650 4750 2    50   Input ~ 0
 col13
-Text GLabel 2650 4650 2    50   Input ~ 0
+Text GLabel 2650 4850 2    50   Input ~ 0
 col14
 Text GLabel 2650 4550 2    50   Input ~ 0
@@
 Text GLabel 2650 4150 2    50   Input ~ 0
 CapsLock
-NoConn ~ 2650 3750
 NoConn ~ 2650 4250
-NoConn ~ 2650 4850
 Text Notes 9250 5500 0    157  ~ 31
 Caps lock LED
@@
 $EndComp
 Text GLabel 10800 1250 1    50   Input ~ 0
-Col14
+col14
 Text GLabel 10000 1250 1    50   Input ~ 0
-Col13
+col13
 Text GLabel 9600 1250 1    50   Input ~ 0
-Col12
+col12
 Text GLabel 9200 1250 1    50   Input ~ 0
-Col11
+col11
 Text GLabel 8800 1250 1    50   Input ~ 0
-Col10
+col10
 Connection ~ 10800 1500
 Wire Wire Line
@@
 	5200 1250 5200 1500
 Connection ~ 4800 1500
-Wire Wire Line
-	4800 1300 4800 1500
 Text GLabel 8400 1250 1    50   Input ~ 0
-Col9
+col9
 Text GLabel 8000 1250 1    50   Input ~ 0
-Col8
+col8
 Text GLabel 7600 1250 1    50   Input ~ 0
-Col7
+col7
 Text GLabel 7200 1250 1    50   Input ~ 0
-Col6
+col6
 Text GLabel 6800 1250 1    50   Input ~ 0
-Col5
+col5
 Text GLabel 6400 1250 1    50   Input ~ 0
-Col4
+col4
 Text GLabel 6000 1250 1    50   Input ~ 0
-Col3
+col3
 Text GLabel 5600 1250 1    50   Input ~ 0
-Col2
+col2
 Text GLabel 5200 1250 1    50   Input ~ 0
-Col1
+col1
 Text GLabel 4800 1250 1    50   Input ~ 0
-Col0
+col0
 Wire Wire Line
 	9950 2250 9900 2250
@@
 	4500 3200 4200 3200
 Text GLabel 4000 2750 0    50   Input ~ 0
-Row1
+row1
 Wire Wire Line
 	4000 2000 4500 2000
 Text GLabel 4000 2000 0    50   Input ~ 0
-Row0
+row0
 $Comp
 L Device:D D1
@@
 $EndComp
 Text GLabel 4000 4250 0    50   Input ~ 0
-Row3
+row3
 Text GLabel 4000 5000 0    50   Input ~ 0
-Row4
+row4
 Text GLabel 4000 3500 0    50   Input ~ 0
-Row2
+row2
 $Comp
 L MX_Alps_Hybrid:MX-NoLED MX74
@@
 	1    0    0    -1
 $EndComp
+NoConn ~ 5350 6700
+NoConn ~ 4950 6700
+Text GLabel 2650 3750 2    50   Input ~ 0
+col7
+Text GLabel 2650 3850 2    50   Input ~ 0
+col9
+Text GLabel 2650 3650 2    50   Input ~ 0
+col5
+Wire Wire Line
+	4800 1250 4800 1500
 $EndSCHEMATC

Commit message: Finished USB-c routing
Parts:
- renumbered R4 to R1, R6 to R2, R5 to R3, R3 to R4, R7 to R5, R8 to R6, R2 to R7, R1 to R8
Changed lines of the file:
@@
 $EndComp
 $Comp
-L Device:R_Small R4
+L Device:R_Small R1
 U 1 1 5F4E9D5C
 P 5400 6300
-F 0 "R4" H 5459 6346 50  0000 L CNN
+F 0 "R1" H 5459 6346 50  0000 L CNN
 F 1 "10k" H 5459 6255 50  0000 L CNN
 F 2 "Resistor_THT:R_Axial_DIN0204_L3.6mm_D1.6mm_P5.08mm_Horizontal" H 5400 6300 50  0001 C CNN
@@
 Connection ~ 3000 7300
 $Comp
-L Device:R_Small R5
+L Device:R_Small R3
 U 1 1 5F4CCFEB
 P 3100 6300
-F 0 "R5" V 2904 6300 50  0000 C CNN
+F 0 "R3" V 2904 6300 50  0000 C CNN
 F 1 "5.1k" V 3000 6300 50  0000 C CNN
 F 2 "Resistor_THT:R_Axial_DIN0204_L3.6mm_D1.6mm_P5.08mm_Horizontal" H 3100 6300 50  0001 C CNN
@@
 	3500 6400 2900 6400
 $Comp
-L Device:R_Small R3
+L Device:R_Small R4
 U 1 1 5F4EB02A
 P 3500 6200
-F 0 "R3" H 3350 6150 50  0000 C CNN
+F 0 "R4" H 3350 6150 50  0000 C CNN
 F 1 "1.5k" H 3350 6250 50  0000 C CNN
 F 2 "Resistor_THT:R_Axial_DIN0204_L3.6mm_D1.6mm_P5.08mm_Horizontal" H 3500 6200 50  0001 C CNN
@@
 	3800 7400 3800 7500
 $Comp
-L Device:R_Small R7
+L Device:R_Small R5
 U 1 1 5F51258F
 P 4000 6400
-F 0 "R7" V 3804 6400 50  0000 C CNN
+F 0 "R5" V 3804 6400 50  0000 C CNN
 F 1 "75" V 3900 6400 50  0000 C CNN
 F 2 "Resistor_THT:R_Axial_DIN0204_L3.6mm_D1.6mm_P5.08mm_Horizontal" H 4000 6400 50  0001 C CNN
@@
 $EndComp
 $Comp
-L Device:R_Small R1
+L Device:R_Small R8
 U 1 1 5F62BAF8
 P 9900 5850
-F 0 "R1" V 9704 5850 50  0000 C CNN
+F 0 "R8" V 9704 5850 50  0000 C CNN
 F 1 "62" V 9795 5850 50  0000 C CNN
 F 2 "Resistor_THT:R_Axial_DIN0204_L3.6mm_D1.6mm_P5.08mm_Horizontal" H 9900 5850 50  0001 C CNN
@@
 $EndComp
 $Comp
-L Device:R_Small R6
+L Device:R_Small R2
 U 1 1 609A6E94
 P 3100 6900
-F 0 "R6" V 2904 6900 50  0000 C CNN
+F 0 "R2" V 2904 6900 50  0000 C CNN
 F 1 "5.1k" V 3000 6900 50  0000 C CNN
 F 2 "Resistor_THT:R_Axial_DIN0204_L3.6mm_D1.6mm_P5.08mm_Horizontal" H 3100 6900 50  0001 C CNN
@@
 $EndComp
 $Comp
-L Device:R_Small R8
+L Device:R_Small R6
 U 1 1 609A7444
 P 4000 6500
-F 0 "R8" V 4100 6500 50  0000 C CNN
+F 0 "R6" V 4100 6500 50  0000 C CNN
 F 1 "75" V 4200 6500 50  0000 C CNN
 F 2 "Resistor_THT:R_Axial_DIN0204_L3.6mm_D1.6mm_P5.08mm_Horizontal" H 4000 6500 50  0001 C CNN
@@
 $EndComp
 $Comp
-L Device:R_Small R2
+L Device:R_Small R7
 U 1 1 609A8C45
 P 6500 6150
-F 0 "R2" V 6300 6150 50  0000 C CNN
+F 0 "R7" V 6300 6150 50  0000 C CNN
 F 1 "1.5k" V 6400 6150 50  0000 C CNN
 F 2 "Resistor_THT:R_Axial_DIN0204_L3.6mm_D1.6mm_P5.08mm_Horizontal" H 6500 6150 50  0001 C CNN

Commit message: More routing
Changed lines of the file:
@@
 	1    0    0    -1
 $EndComp
+Text GLabel 2650 4750 2    50   Input ~ 0
+row3
+Text GLabel 2650 2750 2    50   Input ~ 0
+row1
 Text GLabel 2650 1450 2    50   Input ~ 0
-row3
-Text GLabel 2650 1550 2    50   Input ~ 0
-row1
+col0
 Text GLabel 2650 1650 2    50   Input ~ 0
-col0
-Text GLabel 2650 1750 2    50   Input ~ 0
 col2
 Text GLabel 2650 1850 2    50   Input ~ 0
 col4
+Text GLabel 2650 4650 2    50   Input ~ 0
+row2
 Text GLabel 2650 2650 2    50   Input ~ 0
-row2
-Text GLabel 2650 2750 2    50   Input ~ 0
 row0
-Text GLabel 2650 3450 2    50   Input ~ 0
+Text GLabel 2650 1550 2    50   Input ~ 0
 col1
-Text GLabel 2650 3550 2    50   Input ~ 0
+Text GLabel 2650 1750 2    50   Input ~ 0
 col3
 Text GLabel 2650 2450 2    50   Input ~ 0
@@
 Text GLabel 2650 2550 2    50   Input ~ 0
 B2
-Text GLabel 2650 1950 2    50   Input ~ 0
+Text GLabel 2650 2050 2    50   Input ~ 0
 col6
-Text GLabel 2650 2050 2    50   Input ~ 0
+Text GLabel 2650 3950 2    50   Input ~ 0
 col8
-Text GLabel 2650 2150 2    50   Input ~ 0
+Text GLabel 2650 3750 2    50   Input ~ 0
 col10
-Text GLabel 2650 3950 2    50   Input ~ 0
+Text GLabel 2650 3650 2    50   Input ~ 0
 col11
-Text GLabel 2650 4650 2    50   Input ~ 0
+Text GLabel 2650 3550 2    50   Input ~ 0
 col12
 Text GLabel 2650 2350 2    50   Input ~ 0
 row4
-Text GLabel 2650 4750 2    50   Input ~ 0
+Text GLabel 2650 3450 2    50   Input ~ 0
 col13
 Text GLabel 2650 4850 2    50   Input ~ 0
@@
 NoConn ~ 5350 6700
 NoConn ~ 4950 6700
-Text GLabel 2650 3750 2    50   Input ~ 0
+Text GLabel 2650 2150 2    50   Input ~ 0
 col7
 Text GLabel 2650 3850 2    50   Input ~ 0
 col9
-Text GLabel 2650 3650 2    50   Input ~ 0
+Text GLabel 2650 1950 2    50   Input ~ 0
 col5
 Wire Wire Line

Commit message: Cleaning up top copper layer
Parts:
- J2: symbol USB_C_GCT_USB4085:AVR-ISP-6 -> Ganjing-keyboard-rescue:AVR-ISP-6-USB_C_GCT_USB4085
- MX1, MX10, MX11, MX12, MX13, MX14, MX16, MX17, MX18, MX19, MX2, MX20, MX21, MX22, MX23, MX24, MX25, MX26, MX27, MX28, MX29, MX3, MX30, MX31, MX32, MX33, MX34, MX35, MX36, MX37, MX38, MX39, MX4, MX40, MX41, MX42, MX43, MX44, MX45, MX46, MX47, MX48, MX49, MX5, MX50, MX51, MX52, MX53, MX54, MX55, MX56, MX57, MX58, MX59, MX6, MX60, MX61, MX62, MX63, MX64, MX65, MX66, MX67, MX68, MX69, MX7, MX70, MX71, MX72, MX73, MX74, MX8, MX9: symbol MX_Alps_Hybrid:MX-NoLED -> Ganjing-keyboard-rescue:MX-NoLED-MX_Alps_Hybrid
- S1, S2: symbol dk_Tactile-Switches:1825910-7 -> Ganjing-keyboard-rescue:1825910-7-dk_Tactile-Switches
- U1: symbol MCU_Microchip_ATmega:ATmega32A-PU -> Ganjing-keyboard-rescue:ATmega32A-PU-MCU_Microchip_ATmega
- USB1: symbol USB_C_GCT_USB4085:USB_C_GCT_USB4085 -> Ganjing-keyboard-rescue:USB_C_GCT_USB4085-USB_C_GCT_USB4085
