File: PCB/Ganjing keyboard/Ganjing 65.kicad_pcb (KiCad board)
At the start: 2 copper layers, 304.8 x 122.8 mm, 169 parts, among them J1 Conn_01x04, J2 AVR-ISP-6, SW1 Rotary_Encoder_Switch, U1 ATmega32A-PU, Y1 Crystal

Commit message: Renaming files
Parts:
- renumbered C5 to C1, C3 to C2, C4 to C3, C2 to C4, C1 to C5, S2 to S1, S1 to S2
