File: PCB/Ganjing keyboard/Ganjing 65.sch (KiCad schematic (older format))
At the start: 164 parts, among them J1 Conn_01x04, J2 AVR-ISP-6, SW1 Rotary_Encoder_Switch, U1 ATmega32A-PU, Y1 Crystal

Commit message: Renaming files
Parts:
- J2: symbol Ganjing-keyboard-rescue:AVR-ISP-6-USB_C_GCT_USB4085 -> Ganjing-65-rescue:AVR-ISP-6-USB_C_GCT_USB4085-Ganjing-keyboard-rescue
- MX1, MX10, MX11, MX12, MX13, MX14, MX16, MX17, MX18, MX19, MX2, MX20, MX21, MX22, MX23, MX24, MX25, MX26, MX27, MX28, MX29, MX3, MX30, MX31, MX32, MX33, MX34, MX35, MX36, MX37, MX38, MX39, MX4, MX40, MX41, MX42, MX43, MX44, MX45, MX46, MX47, MX48, MX49, MX5, MX50, MX51, MX52, MX53, MX54, MX55, MX56, MX57, MX58, MX59, MX6, MX60, MX61, MX62, MX63, MX64, MX65, MX66, MX67, MX68, MX69, MX7, MX70, MX71, MX72, MX73, MX74, MX8, MX9: symbol Ganjing-keyboard-rescue:MX-NoLED-MX_Alps_Hybrid -> Ganjing-65-rescue:MX-NoLED-MX_Alps_Hybrid-Ganjing-keyboard-rescue
- S1, S2: symbol Ganjing-keyboard-rescue:1825910-7-dk_Tactile-Switches -> Ganjing-65-rescue:1825910-7-dk_Tactile-Switches-Ganjing-keyboard-rescue
- U1: symbol Ganjing-keyboard-rescue:ATmega32A-PU-MCU_Microchip_ATmega -> Ganjing-65-rescue:ATmega32A-PU-MCU_Microchip_ATmega-Ganjing-keyboard-rescue
- USB1: symbol Ganjing-keyboard-rescue:USB_C_GCT_USB4085-USB_C_GCT_USB4085 -> Ganjing-65-rescue:USB_C_GCT_USB4085-USB_C_GCT_USB4085-Ganjing-keyboard-rescue
- renumbered C5 to C1, C3 to C2, C4 to C3, C2 to C4, C1 to C5
