File: PCB/Ganjing 65/Ganjing 65.sch (KiCad schematic (older format))
At the start: 164 parts, among them J1 Conn_01x04, J2 AVR-ISP-6, SW1 Rotary_Encoder_Switch, U1 ATmega32A-PU, Y1 Crystal

Commit message: Changing some footprints
Parts:
- removed S1: Reset, digikey-footprints:Switch_Tactile_THT_6x6mm, symbol Ganjing-65-rescue:1825910-7-dk_Tactile-Switches-Ganjing-keyboard-rescue
- removed S2: Boot, digikey-footprints:Switch_Tactile_THT_6x6mm, symbol Ganjing-65-rescue:1825910-7-dk_Tactile-Switches-Ganjing-keyboard-rescue
- added S1: Reset, Keyboard:SW_PUSH_6mm, symbol GanJing_components:6mm_tactile_switch
- added S2: Boot, Keyboard:SW_PUSH_6mm, symbol GanJing_components:6mm_tactile_switch
- D1, D10, D11, D12, D13, D14, D15, D16, D17, D18, D19, D2, D20, D21, D22, D23, D24, D25, D26, D27, D28, D29, D3, D30, D31, D32, D33, D34, D35, D36, D37, D38, D39, D4, D40, D41, D42, D43, D44, D45, D46, D47, D48, D49, D5, D50, D51, D52, D53, D54, D55, D56, D57, D58, D59, D6, D60, D61, D62, D63, D64, D65, D66, D67, D7, D8, D9: footprint Diode_THT:D_DO-35_SOD27_P5.08mm_Vertical_AnodeUp -> Keyboard:D_DO-35_SOD27_P5.08mm_Horizontal; symbol Device:D -> GanJing_components:1N4148TR_Diode
- D68, D69: footprint Diode_THT:D_DO-35_SOD27_P5.08mm_Vertical_AnodeUp -> Keyboard:D_DO-35_SOD27_P5.08mm_Horizontal
- J1: footprint Keyboard:ssd1306 128x32 oled -> Keyboard:ssd1306_128x32_oled; symbol Connector_Generic:Conn_01x04 -> GanJing_components:SSD1306_0.91"_OLED
- J2: symbol Ganjing-65-rescue:AVR-ISP-6-USB_C_GCT_USB4085-Ganjing-keyboard-rescue -> GanJing_components:2x3_pin_header
- MX1, MX10, MX11, MX12, MX13, MX14, MX16, MX17, MX18, MX19, MX2, MX20, MX21, MX22, MX23, MX24, MX25, MX26, MX27, MX28, MX29, MX3, MX30, MX31, MX32, MX33, MX34, MX35, MX36, MX37, MX38, MX39, MX4, MX40, MX41, MX42, MX43, MX44, MX45, MX46, MX47, MX48, MX49, MX5, MX50, MX51, MX52, MX53, MX54, MX55, MX56, MX57, MX58, MX59, MX6, MX60, MX61, MX63, MX64, MX65, MX66, MX67, MX69, MX7, MX70, MX71, MX72, MX73, MX8, MX9: symbol Ganjing-65-rescue:MX-NoLED-MX_Alps_Hybrid-Ganjing-keyboard-rescue -> GanJing_components:Cherry_MX_No_LED
- MX62: footprint MX_Only:MXOnly-6.25U-NoLED -> MX_Only:MXOnly-6.25U-ReversedStabilizers-NoLED; symbol Ganjing-65-rescue:MX-NoLED-MX_Alps_Hybrid-Ganjing-keyboard-rescue -> GanJing_components:Cherry_MX_No_LED
- MX68: footprint MX_Only:MXOnly-ISO_NoLED -> MX_Only:MXOnly-ISO-ReversedStabilizers-NoLED; symbol Ganjing-65-rescue:MX-NoLED-MX_Alps_Hybrid-Ganjing-keyboard-rescue -> GanJing_components:Cherry_MX_No_LED
- MX74: footprint MX_Only:MXOnly-7U-NoLED -> MX_Only:MXOnly-7U-ReversedStabilizers-NoLED; symbol Ganjing-65-rescue:MX-NoLED-MX_Alps_Hybrid-Ganjing-keyboard-rescue -> GanJing_components:Cherry_MX_No_LED
- R1, R2, R3, R4, R5, R6, R7: footprint Resistor_THT:R_Axial_DIN0204_L3.6mm_D1.6mm_P5.08mm_Horizontal -> Keyboard:R_Axial_DIN0204_L3.6mm_D1.6mm_P5.08mm_Horizontal
- SW1: symbol Device:Rotary_Encoder_Switch -> GanJing_components:EC11_Rotory_Encoder
- U1: symbol Ganjing-65-rescue:ATmega32A-PU-MCU_Microchip_ATmega-Ganjing-keyboard-rescue -> GanJing_components:ATmega32A-PU
- USB1: footprint Type-C:USB_C_GCT_USB4085 -> Keyboard:USB_C_GCT_USB4085; symbol Ganjing-65-rescue:USB_C_GCT_USB4085-USB_C_GCT_USB4085-Ganjing-keyboard-rescue -> GanJing_components:GCT_USB-c_port
Connections:
- net Boot: now also S2.2
- net GND: now also S1.1, S2.1
- net Reset: now also S1.2
- no-connect marks 9 -> 5
