File: PCB/Ganjing 65/Ganjing 65.kicad_pcb (KiCad board)
At the start: 2 copper layers, 304.8 x 122.8 mm, 169 parts, among them J1 Conn_01x04, J2 AVR-ISP-6, SW1 Rotary_Encoder_Switch, U1 ATmega32A-PU, Y1 Crystal

Commit message: Changing some footprints
Parts:
- R1, R2, R3, R4, R5, R6, R7: footprint Resistor_THT:R_Axial_DIN0204_L3.6mm_D1.6mm_P5.08mm_Horizontal -> Keyboard:R_Axial_DIN0204_L3.6mm_D1.6mm_P5.08mm_Horizontal
- S1, S2: footprint digikey-footprints:Switch_Tactile_THT_6x6mm -> Keyboard:SW_PUSH_6mm
Connections:
- S1 pad 2: Net-(S1-Pad2) -> Reset
- S2 pad 2: Net-(S2-Pad2) -> Boot
Routing:
- net Boot: track 35.2 -> 41.7 mm
Other:
- rule pad_to_mask_clearance: 0.051 -> 0

Commit message: Adding gold lettering
Parts:
- MX31: value Caps Lock -> Standard
- MX43: value Enter -> ANSI Enter
- MX45: value Shift -> ANSI Shift
- MX62: value Space -> 6.25u
- MX69: value Stepped Caps Lock -> Stepped
- MX74: value 7.00u Space -> 7.00u
Other:
- board text added: "GanJing 65"
- board text removed: "GanJing Keyboard"
